File: controller/controller.kicad_sch (KiCad schematic)
At the start: 9 parts, among them U1 Joystick

Commit message: added the pcb design for the controller
Parts:
- Start/stop_wepon1: footprint Button_Switch_THT:SW_TH_Tactile_Omron_B3F-10xx -> Button_Switch_THT:SW_Push_2P1T_Toggle_CK_PVA1xxH4xxxxxxV2
- Stop/start_robot1: footprint Button_Switch_THT:SW_TH_Tactile_Omron_B3F-10xx -> Button_Switch_THT:SW_Push_2P1T_Toggle_CK_PVA1xxH3xxxxxxV2
Changed lines of the file:
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@@
       (effects (font (size 1.27 1.27)) hide)
     )
-    (property "Footprint" "Button_Switch_THT:SW_TH_Tactile_Omron_B3F-10xx" (id 2) (at 134.62 71.12 0)
+    (property "Footprint" "Button_Switch_THT:SW_Push_2P1T_Toggle_CK_PVA1xxH4xxxxxxV2" (id 2) (at 134.62 71.12 0)
       (effects (font (size 1.27 1.27)) hide)
     )
@@
       (effects (font (size 1.27 1.27)) hide)
     )
-    (property "Footprint" "Button_Switch_THT:SW_TH_Tactile_Omron_B3F-10xx" (id 2) (at 134.62 93.98 0)
+    (property "Footprint" "Button_Switch_THT:SW_Push_2P1T_Toggle_CK_PVA1xxH3xxxxxxV2" (id 2) (at 134.62 93.98 0)
       (effects (font (size 1.27 1.27)) hide)
     )
@@
     )
     (path "/198a1923-290d-40d2-bc88-a08e82b80733"
-      (reference "Start/stop_wepon1") (unit 1) (value "SW_MEC_5E") (footprint "Button_Switch_THT:SW_TH_Tactile_Omron_B3F-10xx")
+      (reference "Start/stop_wepon1") (unit 1) (value "SW_MEC_5E") (footprint "Button_Switch_THT:SW_Push_2P1T_Toggle_CK_PVA1xxH4xxxxxxV2")
     )
     (path "/535b76cd-fc12-4f09-acee-3d10d4fb3829"
-      (reference "Stop/start_robot1") (unit 1) (value "SW_MEC_5E") (footprint "Button_Switch_THT:SW_TH_Tactile_Omron_B3F-10xx")
+      (reference "Stop/start_robot1") (unit 1) (value "SW_MEC_5E") (footprint "Button_Switch_THT:SW_Push_2P1T_Toggle_CK_PVA1xxH3xxxxxxV2")
     )
     (path "/744173b2-d2c4-4287-b03e-833300701043"
